File: 2-Design/3-PCB/FlybackConverter/FlybackConverter.kicad_sch (KiCad schematic)
At the start: 44 parts

Commit message: Added test points and connectors. No footprints yet
Parts:
- added Input, Output, PrimaryGND, SecondaryGND, TestPointA, TestPointB, TestPointC, Vo, Vo': Conn_01x01_Female, symbol Connector:Conn_01x01_Female
Connections:
- net GND: now also PrimaryGND.1 (Pin_1)
- net at CIN.1, CIN1.1, CIN2.1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: now also Input.1 (Pin_1)
- net at COUT.1, COUT1.1, COUT2.1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: now also Output.1 (Pin_1), Vo.1 (Pin_1)
- net at COUT.2, COUT1.2, COUT2.2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: now also SecondaryGND.1 (Pin_1)
- net at OPTO.3, RB.2, RC.1: now also TestPointB.1 (Pin_1)
- net at RAC.2, RI.1: now also Vo'.1 (Pin_1)
- net at CP.1, OPTO.2, RJ.1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: now also TestPointA.1 (Pin_1)
- net at CA.2, PWMController.1 (COMP), RA.2: now also TestPointC.1 (Pin_1)
