File: 2-Design/3-PCB/FlybackConverter/FlybackConverter.kicad_sch (KiCad schematic)
At the start: 53 parts

Commit message: i am trying to handle layout
Parts:
- removed DC: D_Zener, symbol Device:D_Zener
- removed Input, Output, PrimaryGND, SecondaryGND: Conn_01x01_Female, symbol Connector:Conn_01x01_Female
- added CVCC2: C, Capacitor_SMD:CP_Elec_8x5.4, symbol Device:C
- added DC1: DZ2S100X0L, Diode_SMD:D_SOD-523, symbol Diode:DZ2S100X0L
- added INPUT1, OUTPUT1: Conn_01x02_Female, TerminalBlock_4Ucon:TerminalBlock_4Ucon_1x02_P3.50mm_Horizontal, symbol Connector:Conn_01x02_Female
- CA1: renamed from CA; footprint (none) -> Capacitor_SMD:C_0805_2012Metric_Pad1.18x1.45mm_HandSolder
- CF1: renamed from CF; footprint (none) -> Capacitor_SMD:C_0805_2012Metric_Pad1.18x1.45mm_HandSolder
- CIN1, CIN2, CIN3, COUT1, COUT2, COUT3: footprint (none) -> Capacitor_SMD:CP_Elec_10x10.5
- CIN4: renamed from CIN; footprint (none) -> Capacitor_SMD:CP_Elec_10x10.5
- COUT4: renamed from COUT; footprint (none) -> Capacitor_SMD:CP_Elec_10x10.5
- CP1: renamed from CP; footprint (none) -> Capacitor_SMD:C_0805_2012Metric_Pad1.18x1.45mm_HandSolder
- CS1, CVCC1: footprint (none) -> Capacitor_SMD:C_0805_2012Metric_Pad1.18x1.45mm_HandSolder
- CSnubber1: renamed from CSnubber; footprint (none) -> Capacitor_SMD:C_2220_5650Metric_Pad1.97x5.40mm_HandSolder
- CT1: renamed from CT; footprint (none) -> Capacitor_SMD:C_0805_2012Metric_Pad1.18x1.45mm_HandSolder
- CVREF1: renamed from CVREF; footprint (none) -> Capacitor_SMD:C_0805_2012Metric_Pad1.18x1.45mm_HandSolder
- CZ1: renamed from CZ; footprint (none) -> Capacitor_SMD:C_0805_2012Metric_Pad1.18x1.45mm_HandSolder
- RC1: renamed from RC; footprint (none) -> Resistor_SMD:R_0805_2012Metric_Pad1.20x1.40mm_HandSolder
- RG1: renamed from RG; footprint (none) -> Resistor_SMD:R_0805_2012Metric_Pad1.20x1.40mm_HandSolder
- TR1: footprint Transformer_THT:Transformer_Breve_TEZ-35x42 -> kutup:sevgi-kafkasi
- TestPointA1: renamed from TestPointA; footprint (none) -> TestPoint:TestPoint_Pad_2.5x2.5mm
- TestPointB1: renamed from TestPointB; footprint (none) -> TestPoint:TestPoint_Pad_2.5x2.5mm
- TestPointC1: renamed from TestPointC; footprint (none) -> TestPoint:TestPoint_Pad_2.5x2.5mm
- Vo'1: renamed from Vo'; footprint (none) -> TestPoint:TestPoint_Pad_2.5x2.5mm
- Vo1: renamed from Vo; footprint (none) -> TestPoint:TestPoint_Pad_2.5x2.5mm
- gave numbers to parts that had none: 2
- renumbered DSnubber to DSnubber1, OPTO to OPTO1, PWMController to PWMController1, RA to RA1, RAC to RAC1, RB to RB1, RCS to RCS1, RE to RE1, RF to RF1, RI to RI1, RJ to RJ1, RK to RK1, RP to RP1, RSnubber to RSnubber1, RT to RT1, RZ to RZ1, TVS_SUBSTITUTE to TVS_SUBSTITUTE1
Connections:
- net GND: now also CVCC2.1, INPUT1.1 (Pin_1)
- net GND1: now also DC1.2 (A)
- net at CIN1.1, CIN2.1, CIN3.1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: now also INPUT1.2 (Pin_2)
- net at COUT1.1, COUT2.1, COUT3.1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: now also OUTPUT1.1 (Pin_1)
- net at COUT1.2, COUT2.2, COUT3.2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: now also OUTPUT1.2 (Pin_2)
- net at RE1.2, RF1.2, RJ1.2: now also DC1.1 (K)
- net at CVCC1.2, PWMController1.7 (VCC), TVS1.1 (K): now also CVCC2.2

Commit message: first tentavie layout
Parts:
- INPUT1, OUTPUT1: footprint TerminalBlock_4Ucon:TerminalBlock_4Ucon_1x02_P3.50mm_Horizontal -> TerminalBlock_Phoenix:TerminalBlock_Phoenix_MKDS-1,5-2-5.08_1x02_P5.08mm_Horizontal
Connections:
- net GND1: now also COUT1.2, COUT2.2, COUT3.2, COUT4.2, OUTPUT1.2 (Pin_2), TR1.6
Changed lines of the file:
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@@
       (effects (font (size 1.27 1.27)) (justify left))
     )
-    (property "Footprint" "TerminalBlock_4Ucon:TerminalBlock_4Ucon_1x02_P3.50mm_Horizontal" (id 2) (at 271.78 48.26 0)
+    (property "Footprint" "TerminalBlock_Phoenix:TerminalBlock_Phoenix_MKDS-1,5-2-5.08_1x02_P5.08mm_Horizontal" (id 2) (at 271.78 48.26 0)
       (effects (font (size 1.27 1.27)) hide)
     )
@@
     (property "Reference" "INPUT1" (id 0) (at 98.425 36.83 0))
     (property "Value" "Conn_01x02_Female" (id 1) (at 98.425 39.37 0))
-    (property "Footprint" "TerminalBlock_4Ucon:TerminalBlock_4Ucon_1x02_P3.50mm_Horizontal" (id 2) (at 97.79 44.45 0)
+    (property "Footprint" "TerminalBlock_Phoenix:TerminalBlock_Phoenix_MKDS-1,5-2-5.08_1x02_P5.08mm_Horizontal" (id 2) (at 97.79 44.45 0)
       (effects (font (size 1.27 1.27)) hide)
     )
@@
     )
     (property "Datasheet" "" (id 3) (at 138.43 71.12 0)
+      (effects (font (size 1.27 1.27)) hide)
+    )
+    (pin "1")
+  )
+  (symbol (lib_id "power:GND1") (at 246.38 54.61 0) (unit 1)
+    (in_bom yes) (on_board yes) (fields_autoplaced)
+    (property "Reference" "#PWR?" (id 0) (at 246.38 60.96 0)
+      (effects (font (size 1.27 1.27)) hide)
+    )
+    (property "Value" "GND1" (id 1) (at 246.38 59.69 0))
+    (property "Footprint" "" (id 2) (at 246.38 54.61 0)
+      (effects (font (size 1.27 1.27)) hide)
+    )
+    (property "Datasheet" "" (id 3) (at 246.38 54.61 0)
       (effects (font (size 1.27 1.27)) hide)
     )
@@
       (reference "#PWR0114") (unit 1) (value "GND") (footprint "")
     )
+    (path "/8516dc0e-3586-40cd-9dde-6aec3044d1d3"
+      (reference "#PWR?") (unit 1) (value "GND1") (footprint "")
+    )
     (path "/35139c98-63bc-4e10-977d-ce5beb339b90"
       (reference "CA1") (unit 1) (value "C") (footprint "Capacitor_SMD:C_0805_2012Metric_Pad1.18x1.45mm_HandSolder")
@@
     )
     (path "/5218f09f-4a8c-4246-bbc5-dc5a647f8801"
-      (reference "INPUT1") (unit 1) (value "Conn_01x02_Female") (footprint "TerminalBlock_4Ucon:TerminalBlock_4Ucon_1x02_P3.50mm_Horizontal")
+      (reference "INPUT1") (unit 1) (value "Conn_01x02_Female") (footprint "TerminalBlock_Phoenix:TerminalBlock_Phoenix_MKDS-1,5-2-5.08_1x02_P5.08mm_Horizontal")
     )
     (path "/4172f9f5-af9c-467d-8404-d5682f0fee29"
@@
     )
     (path "/487a895f-4c3d-4c29-a9ff-8cf89ba54c09"
-      (reference "OUTPUT1") (unit 1) (value "Conn_01x02_Female") (footprint "TerminalBlock_4Ucon:TerminalBlock_4Ucon_1x02_P3.50mm_Horizontal")
+      (reference "OUTPUT1") (unit 1) (value "Conn_01x02_Female") (footprint "TerminalBlock_Phoenix:TerminalBlock_Phoenix_MKDS-1,5-2-5.08_1x02_P5.08mm_Horizontal")
     )
     (path "/9117228d-0af7-4715-ab37-bc92df2921d5"
