File: 2-Design/3-PCB/FlybackConverter/_autosave-FlybackConverter.kicad_sch (KiCad schematic)
At the start: 53 parts

Commit message: Added footprint for the trafo
Parts:
- TR1: footprint Transformer_THT:Transformer_Breve_TEZ-35x42 -> kutup:sevgi-kafkasi
- gave numbers to parts that had none: 2
- renumbered CA to CA1, CF to CF1, CIN to CIN4, COUT to COUT4, CP to CP1, CSnubber to CSnubber1, CT to CT1, CVREF to CVREF1, CZ to CZ1, DC to DC1, DSnubber to DSnubber1, Input to Input1, OPTO to OPTO1, Output to Output1, PWMController to PWMController1, PrimaryGND to PrimaryGND1, RA to RA1, RAC to RAC1, RB to RB1, RC to RC1, RCS to RCS1, RE to RE1, RF to RF1, RG to RG1, RI to RI1, RJ to RJ1, RK to RK1, RP to RP1, RSnubber to RSnubber1, RT to RT1, RZ to RZ1, SecondaryGND to SecondaryGND1, TVS_SUBSTITUTE to TVS_SUBSTITUTE1, TestPointA to TestPointA1, TestPointB to TestPointB1, TestPointC to TestPointC1, Vo' to Vo'1, Vo to Vo1

Commit message: i am trying to handle layout
Parts:
- removed DC1: D_Zener, symbol Device:D_Zener
- removed Input1, Output1, PrimaryGND1, SecondaryGND1: Conn_01x01_Female, symbol Connector:Conn_01x01_Female
- added CVCC2: C, Capacitor_SMD:CP_Elec_8x5.4, symbol Device:C
- added DC1: DZ2S100X0L, Diode_SMD:D_SOD-523, symbol Diode:DZ2S100X0L
- added INPUT1, OUTPUT1: Conn_01x02_Female, TerminalBlock_Phoenix:TerminalBlock_Phoenix_MKDS-1,5-2-5.08_1x02_P5.08mm_Horizontal, symbol Connector:Conn_01x02_Female
- CA1, CF1, CP1, CS1, CT1, CVCC1, CVREF1, CZ1: footprint (none) -> Capacitor_SMD:C_0805_2012Metric_Pad1.18x1.45mm_HandSolder
- CIN1, CIN2, CIN3, CIN4, COUT1, COUT2, COUT3, COUT4: footprint (none) -> Capacitor_SMD:CP_Elec_10x10.5
- CSnubber1: footprint (none) -> Capacitor_SMD:C_2220_5650Metric_Pad1.97x5.40mm_HandSolder
- RC1, RG1: footprint (none) -> Resistor_SMD:R_0805_2012Metric_Pad1.20x1.40mm_HandSolder
- TestPointA1, TestPointB1, TestPointC1, Vo'1, Vo1: footprint (none) -> TestPoint:TestPoint_Pad_2.5x2.5mm
Connections:
- net GND: now also CVCC2.1, INPUT1.1 (Pin_1)
- net GND1: now also DC1.2 (A)
- net at CIN1.1, CIN2.1, CIN3.1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: now also INPUT1.2 (Pin_2)
- net at COUT1.1, COUT2.1, COUT3.1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: now also OUTPUT1.1 (Pin_1)
- net at COUT1.2, COUT2.2, COUT3.2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: now also OUTPUT1.2 (Pin_2)
- net at RE1.2, RF1.2, RJ1.2: now also DC1.1 (K)
- net at CVCC1.2, PWMController1.7 (VCC), TVS1.1 (K): now also CVCC2.2
